File: 4-bit-rca.kicad_pcb (KiCad board)
At the start: 2 copper layers, 115.6 x 80 mm, 25 parts, among them J1 Cin, J2 Cout, SW1 SW_SPST, SW2 SW_SPST, SW3 SW_SPST, SW4 SW_SPST, SW5 SW_SPST, SW6 SW_SPST, SW7 SW_SPST, SW8 SW_SPST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

Commit message: redo
Parts:
- moved U6 2.54 mm to (78.7, 149.9)
Routing:
- net Net-(R1-Pad2): track 169.4 -> 90.5 mm, vias 0 -> 2
- net Net-(BT1--): track 274.2 -> 210.0 mm
- net Net-(SW1-B): track 115.2 -> 79.2 mm, vias 2 -> 5
- net Net-(U4-Pad5): track 91.3 -> 55.9 mm, vias 3 -> 6
- net Net-(SW1-A): track 322.0 -> 286.9 mm, vias 6 -> 17
- net Net-(U3-Pad6): track 84.7 -> 51.9 mm
- net Net-(J1-Pin_1): track 102.4 -> 72.4 mm, vias 2 -> 5
- net Net-(SW4-B): track 134.7 -> 106.8 mm, vias 0 -> 6
- net Net-(SW7-B): track 90.3 -> 115.7 mm, vias 2 -> 9
- net Net-(SW8-B): track 110.1 -> 89.0 mm, vias 2 -> 7
- net Net-(U3-Pad10): track 31.3 -> 14.0 mm
- net Net-(SW5-B): track 106.8 -> 90.1 mm, vias 1 -> 5
- net Net-(SW3-B): track 130.9 -> 144.8 mm, vias 0 -> 7
- net Net-(U3-Pad12): track 52.4 -> 39.4 mm, vias 2 -> 3
- net Net-(SW6-B): track 74.5 -> 86.0 mm, vias 2 -> 5
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
Commit message: aoisjdojoasd
Parts:
- removed SW2, SW3, SW4, SW5, SW6, SW7, SW8: SW_SPST, Button_Switch_THT:SW_PUSH_6mm
- added R10: 10k, Resistor_THT:R_Axial_DIN0207_L6.3mm_D2.5mm_P10.16mm_Horizontal, F.Cu at (132.3, 106.4)
- added R11: 10k, Resistor_THT:R_Axial_DIN0207_L6.3mm_D2.5mm_P10.16mm_Horizontal, F.Cu at (128.3, 106.4)
- added R12: 10k, Resistor_THT:R_Axial_DIN0207_L6.3mm_D2.5mm_P10.16mm_Horizontal, F.Cu at (124.1, 106.4)
- added R5: 10k, Resistor_THT:R_Axial_DIN0207_L6.3mm_D2.5mm_P10.16mm_Horizontal, F.Cu at (152.6, 106.4)
- added R6: 10k, Resistor_THT:R_Axial_DIN0207_L6.3mm_D2.5mm_P10.16mm_Horizontal, F.Cu at (148.5, 106.5)
- added R7: 10k, Resistor_THT:R_Axial_DIN0207_L6.3mm_D2.5mm_P10.16mm_Horizontal, F.Cu at (144.5, 106.4)
- added R8: 10k, Resistor_THT:R_Axial_DIN0207_L6.3mm_D2.5mm_P10.16mm_Horizontal, F.Cu at (140.4, 106.4)
- added R9: 10k, Resistor_THT:R_Axial_DIN0207_L6.3mm_D2.5mm_P10.16mm_Horizontal, F.Cu at (136.4, 106.4)
- SW1: value SW_SPST -> SW_DIP_x08; footprint Button_Switch_THT:SW_PUSH_6mm -> Button_Switch_SMD:SW_DIP_SPSTx08_Slide_9.78x22.5mm_W8.61mm_P2.54mm
- U6: footprint Package_TO_SOT_THT:TO-92 -> Package_TO_SOT_THT:TO-220-3_Vertical
- moved BT1 129.7 mm to (199.4, 130.8)
- moved J1 129.3 mm to (199.4, 114.3)
- moved J2 129.3 mm to (199.4, 120.7)
- moved U6 109.6 mm to (186.7, 130.8)
- moved SW1 65.3 mm to (142.2, 131.6)
- moved U1 39.6 mm to (110.2, 62.0)
- moved U2 39.6 mm to (130.6, 62.0)
- moved U3 39.6 mm to (149.6, 62.0)
- moved U5 39.6 mm to (190.3, 62.0)
- moved U4 39.6 mm to (168.7, 62.0)
- moved D1 29.5 mm to (160.0, 111.8)
- moved D2 29.5 mm to (167.6, 111.8)
- moved D3 29.5 mm to (175.4, 111.8)
- moved D4 29.5 mm to (182.9, 111.8)
- moved R1 29.5 mm to (165.1, 104.1)
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Connections:
- SW1 pad 1: Net-(SW1-A) -> Net-(U1E-VCC)
- SW1 pad 2: Net-(SW1-B) -> Net-(U1E-VCC)
- U1 pad 1: Net-(SW1-B) -> Net-(R12-Pad1)
- U1 pad 14: Net-(SW1-A) -> Net-(U1E-VCC)
- U1 pad 2: Net-(SW5-B) -> Net-(R8-Pad1)
- U2 pad 14: Net-(SW1-A) -> Net-(U1E-VCC)
- U2 pad 4: Net-(SW1-B) -> Net-(R12-Pad1)
- U2 pad 5: Net-(SW5-B) -> Net-(R5-Pad1)
- U3 pad 14: Net-(SW1-A) -> Net-(U1E-VCC)
- U4 pad 10: Net-(SW8-B) -> Net-(R5-Pad1)
- U4 pad 14: Net-(SW1-A) -> Net-(U1E-VCC)
- U5 pad 10: Net-(SW8-B) -> Net-(R5-Pad1)
- U5 pad 14: Net-(SW1-A) -> Net-(U1E-VCC)
- U6 pad 3: Net-(SW1-A) -> Net-(U1E-VCC)
Routing:
- net Net-(SW1-A): track 286.9 -> 0.00 mm, vias 17 -> 0
- net Net-(U1E-VCC): track 0.00 -> 254.7 mm, vias 0 -> 14
- net Net-(R5-Pad1): track 0.00 -> 99.6 mm, vias 0 -> 9
- net Net-(SW5-B): track 90.1 -> 0.00 mm, vias 5 -> 0
- net Net-(SW8-B): track 89.0 -> 0.00 mm, vias 7 -> 0
- net Net-(R12-Pad1): track 0.00 -> 86.9 mm, vias 0 -> 4
- net Net-(R8-Pad1): track 0.00 -> 86.6 mm, vias 0 -> 7
- net Net-(J1-Pin_1): track 72.4 -> 154.0 mm, vias 5 -> 9
- net Net-(SW1-B): track 79.2 -> 0.00 mm, vias 5 -> 0
- net Net-(R2-Pad2): track 85.4 -> 67.5 mm, vias 2 -> 1
- net Net-(R1-Pad2): track 90.5 -> 75.8 mm
- net Net-(R12-Pad2): track 0.00 -> 14.5 mm
- net Net-(R3-Pad2): track 28.3 -> 42.4 mm, vias 1 -> 3
- net Net-(R11-Pad2): track 0.00 -> 13.9 mm
- net Net-(R10-Pad2): track 0.00 -> 13.2 mm
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Other:
- board outline removed

Commit message: a
Parts:
- removed J2: Cout, Connector_PinHeader_2.54mm:PinHeader_1x01_P2.54mm_Vertical
- added D5: LED, LED_THT:LED_D5.0mm, F.Cu at (193.9, 112.5)
- added R13: 360, Resistor_THT:R_Axial_DIN0207_L6.3mm_D2.5mm_P10.16mm_Horizontal, F.Cu at (190.5, 101.6)
- J1: value Cin -> CIN & COUT; footprint Connector_PinHeader_2.54mm:PinHeader_1x01_P2.54mm_Vertical -> Connector_PinHeader_2.54mm:PinHeader_1x02_P2.54mm_Vertical
- SW1: footprint Button_Switch_SMD:SW_DIP_SPSTx08_Slide_9.78x22.5mm_W8.61mm_P2.54mm -> Button_Switch_THT:SW_DIP_SPSTx08_Slide_6.7x21.88mm_W7.62mm_P2.54mm_LowProfile
- moved SW1 8.75 mm to (134.6, 135.9)
- moved J1 6.35 mm to (199.4, 120.7), turned to 180 degrees
Connections:
- U1 pad 5: Net-(J1-Pin_1) -> Net-(J1-Pin_2)
- U2 pad 1: Net-(J1-Pin_1) -> Net-(J1-Pin_2)
- U3 pad 11: Net-(J2-Pin_1) -> Net-(J1-Pin_1)
Routing:
- net Net-(J1-Pin_2): track 0.00 -> 157.8 mm, vias 0 -> 9
- net Net-(J2-Pin_1): track 98.2 -> 0.00 mm, vias 4 -> 0
- net Net-(R5-Pad1): track 99.6 -> 167.5 mm, vias 9 -> 11
- net Net-(J1-Pin_1): track 154.0 -> 118.4 mm, vias 9 -> 4
- net Net-(D5-A): track 0.00 -> 13.4 mm
- net Net-(R8-Pad1): track 86.6 -> 80.1 mm
- net Net-(U1E-VCC): track 254.7 -> 248.3 mm, vias 14 -> 10
- net Net-(BT1--): track 200.2 -> 204.7 mm
- net Net-(R9-Pad2): track 12.6 -> 14.1 mm
- net Net-(R6-Pad2): track 10.7 -> 12.2 mm
- net Net-(R11-Pad2): track 13.9 -> 15.4 mm
- net Net-(R8-Pad2): track 12.0 -> 13.5 mm
- net Net-(R12-Pad2): track 14.5 -> 16.0 mm
- net Net-(R7-Pad2): track 11.8 -> 13.3 mm
- net Net-(R10-Pad2): track 13.2 -> 14.7 mm
Other:
- board outline added: 97.8 x 92.7 mm
- board text added: "Cin"
- board text added: "Cout"
- board text added: "JLCJLCJLCJLC"

Commit message: a
Parts:
- moved R6 0.25 mm to (148.6, 106.7)
- moved R11 0.25 mm to (128.4, 106.6)
- moved R7 0.25 mm to (144.6, 106.6)
- moved R9 0.25 mm to (136.5, 106.6)
- moved R12 0.25 mm to (124.2, 106.7)
- moved R10 0.25 mm to (132.4, 106.6)
- moved R5 0.25 mm to (152.7, 106.6)
- moved R8 0.25 mm to (140.5, 106.6)
Connections:
- R10 pad 2: Net-(R10-Pad2) -> Net-(BT1--)
- R11 pad 2: Net-(R11-Pad2) -> Net-(BT1--)
- R12 pad 2: Net-(R12-Pad2) -> Net-(BT1--)
- R5 pad 2: Net-(R5-Pad2) -> Net-(BT1--)
- R6 pad 2: Net-(R6-Pad2) -> Net-(BT1--)
- R7 pad 2: Net-(R7-Pad2) -> Net-(BT1--)
- R8 pad 2: Net-(R8-Pad2) -> Net-(BT1--)
- R9 pad 2: Net-(R9-Pad2) -> Net-(BT1--)
- SW1 pad 10: Net-(R6-Pad2) -> Net-(R7-Pad1)
- SW1 pad 11: Net-(R7-Pad2) -> Net-(R9-Pad1)
- SW1 pad 12: Net-(R8-Pad2) -> Net-(R11-Pad1)
- SW1 pad 13: Net-(R9-Pad2) -> Net-(R6-Pad1)
- SW1 pad 14: Net-(R10-Pad2) -> Net-(R8-Pad1)
- SW1 pad 15: Net-(R11-Pad2) -> Net-(R10-Pad1)
- SW1 pad 16: Net-(R12-Pad2) -> Net-(R12-Pad1)
- SW1 pad 9: Net-(R5-Pad2) -> Net-(R5-Pad1)
- U1 pad 12: Net-(R11-Pad1) -> Net-(R10-Pad1)
- U1 pad 13: Net-(R7-Pad1) -> Net-(R9-Pad1)
- U1 pad 2: Net-(R8-Pad1) -> Net-(R11-Pad1)
- U2 pad 10: Net-(R7-Pad1) -> Net-(R9-Pad1)
- U2 pad 5: Net-(R5-Pad1) -> Net-(R11-Pad1)
- U2 pad 9: Net-(R11-Pad1) -> Net-(R10-Pad1)
- U4 pad 1: Net-(R10-Pad1) -> Net-(R8-Pad1)
- U4 pad 2: Net-(R6-Pad1) -> Net-(R7-Pad1)
- U4 pad 9: Net-(R9-Pad1) -> Net-(R6-Pad1)
- U5 pad 4: Net-(R10-Pad1) -> Net-(R8-Pad1)
- U5 pad 5: Net-(R6-Pad1) -> Net-(R7-Pad1)
- U5 pad 9: Net-(R9-Pad1) -> Net-(R6-Pad1)
Routing:
- net Net-(R7-Pad1): track 87.4 -> 177.0 mm, vias 7 -> 12
- net Net-(R11-Pad1): track 91.5 -> 166.2 mm, vias 4 -> 8
- net Net-(BT1--): track 204.7 -> 257.2 mm, vias 10 -> 11
- net Net-(R10-Pad1): track 142.5 -> 90.3 mm, vias 7 -> 5
- net Net-(R5-Pad1): track 167.5 -> 122.8 mm, vias 11 -> 9
- net Net-(R8-Pad1): track 80.1 -> 118.8 mm, vias 7 -> 3
- net Net-(R12-Pad1): track 86.9 -> 117.3 mm, vias 4 -> 5
- net Net-(R12-Pad2): track 16.0 -> 0.00 mm
- net Net-(R11-Pad2): track 15.4 -> 0.00 mm
- net Net-(R10-Pad2): track 14.7 -> 0.00 mm
- net Net-(R9-Pad2): track 14.1 -> 0.00 mm
- net Net-(R8-Pad2): track 13.5 -> 0.00 mm
- net Net-(R7-Pad2): track 13.3 -> 0.00 mm
- net Net-(R6-Pad1): track 121.4 -> 133.8 mm, vias 11 -> 12
- net Net-(R6-Pad2): track 12.2 -> 0.00 mm
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
Commit message: a
Routing:
- net Net-(R6-Pad1): track 133.8 -> 128.7 mm, vias 12 -> 10
Changed lines of the file:
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@@
   (segment (start 186.436 86.106) (end 172.974 86.106) (width 0.5) (layer "B.Cu") (net 27))
   (segment (start 162.306 89.298) (end 161.98 88.972) (width 0.5) (layer "F.Cu") (net 28))
-  (segment (start 185.166 72.136) (end 185.166 70.866) (width 0.5) (layer "F.Cu") (net 28))
   (segment (start 148.506 101.176) (end 149.606 100.076) (width 0.5) (layer "F.Cu") (net 28))
   (segment (start 173.99 71.12) (end 173.99 72.39) (width 0.5) (layer "F.Cu") (net 28))
@@
   (segment (start 142.24 113.03) (end 148.59 106.68) (width 0.5) (layer "F.Cu") (net 28))
   (via (at 162.306 88.646) (size 0.8) (drill 0.4) (layers "F.Cu" "B.Cu") (net 28))
-  (via (at 185.166 70.866) (size 0.8) (drill 0.4) (layers "F.Cu" "B.Cu") (net 28))
   (via (at 178.816 73.406) (size 0.8) (drill 0.4) (layers "F.Cu" "B.Cu") (net 28))
   (via (at 162.306 100.076) (size 0.8) (drill 0.4) (layers "F.Cu" "B.Cu") (net 28))
@@
   (via (at 195.326 74.676) (size 0.8) (drill 0.4) (layers "F.Cu" "B.Cu") (net 28))
   (via (at 181.356 88.646) (size 0.8) (drill 0.4) (layers "F.Cu" "B.Cu") (net 28))
-  (via (at 185.166 72.136) (size 0.8) (drill 0.4) (layers "F.Cu" "B.Cu") (net 28))
   (via (at 181.356 70.866) (size 0.8) (drill 0.4) (layers "F.Cu" "B.Cu") (net 28))
   (via (at 149.606 100.076) (size 0.8) (drill 0.4) (layers "F.Cu" "B.Cu") (net 28))
   (via (at 173.99 71.12) (size 0.8) (drill 0.4) (layers "F.Cu" "B.Cu") (net 28))
-  (segment (start 185.166 70.866) (end 182.626 70.866) (width 0.5) (layer "B.Cu") (net 28))
-  (segment (start 181.356 70.866) (end 182.626 70.866) (width 0.5) (layer "B.Cu") (net 28))
-  (segment (start 185.171 72.131) (end 185.166 72.136) (width 0.5) (layer "B.Cu") (net 28))
   (segment (start 174.244 70.866) (end 173.99 71.12) (width 0.5) (layer "B.Cu") (net 28))
   (segment (start 162.306 88.646) (end 181.356 88.646) (width 0.5) (layer "B.Cu") (net 28))
